File: PAF-hw/PAF-hw_Electrical/PAF-hw_Electrical_Project/Stepper_Driver.kicad_sch (KiCad schematic)
At the start: 10 parts, among them IC4 DRV8425PWPR

Commit message: Added camera circuit to schematic.
Parts:
- added C27, C28: 22uF, CAPC2012X95N, symbol SamacSys_Parts:CL21A226KPCLRNC
Connections:
- net 12V_UNREG: now also C27.1, C28.1
- net GND: now also C27.2, C28.2
Other:
- moved on the sheet: C15, C18, C19, C20, C8, IC4
